File: parts/_74xx/_74LS595.kicad_sch (KiCad schematic)
At the start: 25 parts, among them U1 INV, U10 BUF_G, U11 D_LATCH, U12 D_LATCH, U13 BUF_G, U14 D_LATCH, U15 D_LATCH, U16 BUF_G, U17 D_LATCH, U18 D_LATCH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

Commit message: Added/Updated parts.
Connections:
- no-connect marks 15 -> 16
Changed lines of the file:
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@@
+	)
+	(no_connect
+		(at 210.82 41.91)
 	)
 	(no_connect
